Commit message: Updated

File: ros2_ws/install/transport_bot/share/transport_bot/urdf/transport_bot.urdf.xacro (robot description, xacro)
@@ -2,4 +2,5 @@
 <robot name="transport_bot" xmlns:xacro="http://ros.org/wiki/xacro">
   <xacro:property name="wheel_radius" value="0.05"/>
+  <xacro:property name="wheel_diameter" value="0.10"/>
   <xacro:property name="wheel_width" value="0.02"/>
   <xacro:property name="base_length" value="0.4"/>
@@ -60,4 +61,7 @@
   <!-- Rear Right -->
   <xacro:wheel name="wheel_rr" x="-${base_length/2}" y="-${base_width/2}"/>
+<!-- Differential Drive (For Motion)a kinematic model used for robots that move
+using two independently driven wheels, typically placed on either side of the chassis.
+-->
 <gazebo>
   <plugin name="diff_drive" filename="libgazebo_ros_diff_drive.so">
@@ -77,3 +81,72 @@
   </plugin>
 </gazebo>
+<!-- Depth Camera Link -->
+<link name="depth_camera_link">
+  <visual>
+    <geometry>
+      <box size="0.05 0.05 0.05"/>
+    </geometry>
+    <material name="black">
+      <color rgba="0 0 0 1"/>
+    </material>
+  </visual>
+  <collision>
+    <geometry>
+      <box size="0.05 0.05 0.05"/>
+    </geometry>
+  </collision>
+  <inertial>
+    <mass value="0.2"/>
+    <origin xyz="0 0 0" rpy="0 0 0"/>
+    <inertia ixx="0.01" ixy="0.0" ixz="0.0" iyy="0.01" iyz="0.0" izz="0.01"/>
+  </inertial>
+</link>
+<joint name="depth_camera_joint" type="fixed">
+  <parent link="base_link"/>
+  <child link="depth_camera_link"/>
+  <origin xyz="0 0 ${base_height/2 + 0.2}" rpy="0 0 0"/>
+</joint>
+<gazebo reference="depth_camera_link">
+  <sensor name="depth_camera" type="depth">
+    <always_on>true</always_on>
+    <update_rate>30.0</update_rate>
+    <visualize>true</visualize>
+    <camera>
+      <horizontal_fov>1.3962634</horizontal_fov>
+      <image>
+        <width>640</width>
+        <height>480</height>
+        <format>R8G8B8</format>
+      </image>
+      <clip>
+        <near>0.05</near>
+        <far>10.0</far>
+      </clip>
+    </camera>
+    <plugin name="depth_camera_link_controller" filename="libgazebo_ros_openni_kinect.so">
+      <baseline>0.2</baseline>
+      <alwaysOn>true</alwaysOn>
+      <updateRate>1.0</updateRate>
+      <cameraName>depth_camera_ir</cameraName>
+      <imageTopicName>/depth_camera/color/image_raw</imageTopicName>
+      <cameraInfoTopicName>/depth_camera/color/camera_info</cameraInfoTopicName>
+      <depthImageTopicName>/depth_camera/depth/image_raw</depthImageTopicName>
+      <depthImageInfoTopicName>/depth_camera/depth/camera_info</depthImageInfoTopicName>
+      <pointCloudTopicName>/depth_camera/depth/points</pointCloudTopicName>
+      <frameName>base_link</frameName>
+      <pointCloudCutoff>0.5</pointCloudCutoff>
+      <pointCloudCutoffMax>3.0</pointCloudCutoffMax>
+      <distortionK1>0.00000001</distortionK1>
+      <distortionK2>0.00000001</distortionK2>
+      <distortionK3>0.00000001</distortionK3>
+      <distortionT1>0.00000001</distortionT1>
+      <distortionT2>0.00000001</distortionT2>
+      <CxPrime>0</CxPrime>
+      <Cx>0</Cx>
+      <Cy>0</Cy>
+      <focalLength>0</focalLength>
+      <hackBaseline>0</hackBaseline>
+    </plugin>
+  </sensor>
+</gazebo>
 </robot>
